File: hardware/YuEEG_8CH_RevH_Stack/power/YuEEG_H_POWER.kicad_pcb (KiCad board)
At the start: 2 copper layers, 34 x 18 mm, 21 parts

Commit message: Refine Rev H module legends and USB return paths
Other:
- board text added: "1S POWER"
- board text added: "PROTECT"
